File: PCB FILES/vBoard/vBoard.kicad_pcb (KiCad board)
At the start: 2 copper layers, 413.5 x 159.5 mm, 203 parts, among them SW1 SW_Push, SW10 SW_Push, SW11 SW_Push, SW12 SW_Push, SW13 SW_Push, SW14 SW_Push, SW15 SW_Push, SW16 SW_Push, SW17 SW_Push, SW18 SW_Push, SW19 SW_Push, SW2 SW_Push, SW20 SW_Push, SW21 SW_Push, SW22 SW_Push, SW23 SW_Push, SW24 SW_Push, SW25 SW_Push, SW26 SW_Push, SW27 SW_Push, SW28 SW_Push, SW29 SW_Push, SW3 SW_Push, SW30 SW_Push, SW31 SW_Push, SW32 SW_Push, SW33 SW_Push, SW34 SW_Push, SW35 SW_Push, SW36 SW_Push, SW37 SW_Push, SW38 SW_Push, SW39 SW_Push, SW4 SW_Push, SW40 SW_Push, SW41 SW_Push, SW42 SW_Push, SW43 SW_Push, SW44 SW_Push, SW45 SW_Push, SW46 SW_Push, SW47 SW_Push, SW48 SW_Push, SW49 SW_Push, SW5 SW_Push, SW50 SW_Push, SW51 SW_Push, SW52 SW_Push, SW53 SW_Push, SW54 SW_Push, SW55 SW_Push, SW56 SW_Push, SW57 SW_Push, SW58 SW_Push, SW59 SW_Push, SW6 SW_Push, SW60 SW_Push, SW61 SW_Push, SW62 SW_Push, SW63 SW_Push, SW64 SW_Push, SW65 SW_Push, SW66 SW_Push, SW67 SW_Push, SW68 SW_Push, SW69 SW_Push, SW7 SW_Push, SW70 SW_Push, SW71 SW_Push, SW72 SW_Push, SW73 SW_Push, SW74 SW_Push, SW75 SW_Push, SW76 SW_Push, SW77 SW_Push, SW78 SW_Push, SW79 SW_Push, SW8 SW_Push, SW80 SW_Push, SW81 SW_Push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

Commit message: journaling kicad. Will work on cad after pcb.
Parts:
- moved D98 2.60 mm to (419.1, 90.5)
Connections:
- A1 pad 7: /Row 5 -> /COL9
- D85 pad 1: /Row 5 -> /COL9
- D86 pad 1: /Row 5 -> /COL9
- D87 pad 1: /Row 5 -> /COL9
- D88 pad 1: /Row 5 -> /COL9
- D89 pad 1: /Row 5 -> /COL9
- D90 pad 1: /Row 5 -> /COL9
- D91 pad 1: /Row 5 -> /COL9
- D93 pad 1: /Row 5 -> /COL9
- D94 pad 1: /Row 5 -> /COL9
- D95 pad 1: /Row 5 -> /COL9
- D96 pad 1: /Row 5 -> /COL9
- D97 pad 1: /Row 5 -> /COL9
- D98 pad 1: /Row 5 -> /COL9
Routing:
- net /COL9: track 0.00 -> 924.6 mm
- net /Row 1: track 0.00 -> 491.4 mm
- net /Row 4: track 0.00 -> 449.8 mm
- net /Row 2: track 0.00 -> 449.2 mm
- net /Row 3: track 0.00 -> 441.5 mm
- net /Fn Row: track 0.00 -> 408.8 mm
- net Net-(D88-A): track 0.00 -> 74.8 mm
- net /ROT0: track 0.00 -> 53.8 mm
- net Net-(A1-GPIO28_ADC2): track 0.00 -> 52.4 mm
- net Net-(D69-A): track 0.00 -> 31.2 mm
- net Net-(D65-A): track 0.00 -> 31.2 mm
- net Net-(D30-A): track 0.00 -> 31.2 mm
- net Net-(A1-GND-Pad13): track 0.00 -> 27.1 mm
- net Net-(D68-A): track 0.00 -> 22.4 mm
- net /COL17: track 0.00 -> 22.1 mm
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
Commit message: EH
Routing:
- net /COL12: track 0.00 -> 134.1 mm
- net /COL10: track 0.00 -> 133.7 mm
- net /COL9: track 924.6 -> 1057.8 mm
- net /COL8: track 0.00 -> 129.2 mm
- net /COL1: track 0.00 -> 125.5 mm
- net /COL2: track 0.00 -> 123.7 mm
- net /COL5: track 0.00 -> 123.5 mm
- net /COL14: track 0.00 -> 115.4 mm
- net /COL11: track 0.00 -> 113.7 mm
- net /COL0: track 0.00 -> 113.6 mm
- net /COL16: track 0.00 -> 108.7 mm
- net /COL15: track 0.00 -> 108.7 mm
- net /COL7: track 0.00 -> 103.6 mm
- net /COL6: track 0.00 -> 103.5 mm
- net /COL3: track 0.00 -> 99.5 mm
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
Commit message: Journaling and got some more work done.
Parts:
- added H1: MountingHole, MountingHole:MountingHole_3.2mm_M3, F.Cu at (43.7, 203.2)
- added H10: MountingHole, MountingHole:MountingHole_3.2mm_M3, F.Cu at (332.6, 54.8)
- added H11: MountingHole, MountingHole:MountingHole_3.2mm_M3, F.Cu at (414.3, 55.6)
- added H12: MountingHole, MountingHole:MountingHole_3.2mm_M3, F.Cu at (438.1, 171.4)
- added H2: MountingHole, MountingHole:MountingHole_3.2mm_M3, F.Cu at (139.7, 203.2)
- added H3: MountingHole, MountingHole:MountingHole_3.2mm_M3, F.Cu at (235.7, 203.2)
- added H4: MountingHole, MountingHole:MountingHole_3.2mm_M3, F.Cu at (332.6, 203.2)
- added H5: MountingHole, MountingHole:MountingHole_3.2mm_M3, F.Cu at (449.2, 203.2)
- added H6: MountingHole, MountingHole:MountingHole_3.2mm_M3, F.Cu at (43.7, 132.5)
- added H7: MountingHole, MountingHole:MountingHole_3.2mm_M3, F.Cu at (48.4, 54.0)
- added H8: MountingHole, MountingHole:MountingHole_3.2mm_M3, F.Cu at (138.9, 54.8)
- added H9: MountingHole, MountingHole:MountingHole_3.2mm_M3, F.Cu at (235.7, 54.8)
Routing:
- net /COL4: track 99.5 -> 538.8 mm, vias 0 -> 2
- net /COL0: track 113.6 -> 533.7 mm
- net /COL3: track 99.5 -> 497.8 mm, vias 0 -> 2
- net /COL1: track 125.5 -> 521.2 mm, vias 0 -> 2
- net /COL5: track 123.5 -> 509.9 mm, vias 0 -> 2
- net /COL6: track 103.5 -> 489.4 mm, vias 0 -> 3
- net /COL2: track 123.7 -> 497.3 mm, vias 0 -> 2
- net /COL7: track 103.6 -> 441.9 mm, vias 0 -> 3
- net /COL8: track 129.2 -> 431.6 mm, vias 0 -> 3
- net /COL11: track 113.7 -> 387.4 mm, vias 0 -> 2
- net /COL9: track 1057.8 -> 1313.7 mm
- net /COL10: track 133.7 -> 380.1 mm, vias 0 -> 1
- net /COL12: track 134.1 -> 361.7 mm, vias 0 -> 1
- net /COL13: track 86.9 -> 295.1 mm, vias 0 -> 3
- net /COL14: track 115.4 -> 310.0 mm, vias 0 -> 3
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- added copper zone on B.Cu, net Net-(A1-GND-Pad13)

Commit message: DRC fixes.
Routing:
- net /Row 4: track 449.8 -> 470.9 mm, vias 0 -> 2
- net /Row 3: track 441.5 -> 438.3 mm
- net /ROT0: track 53.8 -> 54.2 mm, vias 0 -> 2
- net /COL6: track 489.4 -> 489.5 mm, vias 3 -> 4
