File: PCB FILES/vBoard/vBoard.kicad_pcb (KiCad board)
At the start: 2 copper layers, 413.5 x 159.5 mm, 215 parts, among them SW1 SW_Push, SW10 SW_Push, SW11 SW_Push, SW12 SW_Push, SW13 SW_Push, SW14 SW_Push, SW15 SW_Push, SW16 SW_Push, SW17 SW_Push, SW18 SW_Push, SW19 SW_Push, SW2 SW_Push, SW20 SW_Push, SW21 SW_Push, SW22 SW_Push, SW23 SW_Push, SW24 SW_Push, SW25 SW_Push, SW26 SW_Push, SW27 SW_Push, SW28 SW_Push, SW29 SW_Push, SW3 SW_Push, SW30 SW_Push, SW31 SW_Push, SW32 SW_Push, SW33 SW_Push, SW34 SW_Push, SW35 SW_Push, SW36 SW_Push, SW37 SW_Push, SW38 SW_Push, SW39 SW_Push, SW4 SW_Push, SW40 SW_Push, SW41 SW_Push, SW42 SW_Push, SW43 SW_Push, SW44 SW_Push, SW45 SW_Push, SW46 SW_Push, SW47 SW_Push, SW48 SW_Push, SW49 SW_Push, SW5 SW_Push, SW50 SW_Push, SW51 SW_Push, SW52 SW_Push, SW53 SW_Push, SW54 SW_Push, SW55 SW_Push, SW56 SW_Push, SW57 SW_Push, SW58 SW_Push, SW59 SW_Push, SW6 SW_Push, SW60 SW_Push, SW61 SW_Push, SW62 SW_Push, SW63 SW_Push, SW64 SW_Push, SW65 SW_Push, SW66 SW_Push, SW67 SW_Push, SW68 SW_Push, SW69 SW_Push, SW7 SW_Push, SW70 SW_Push, SW71 SW_Push, SW72 SW_Push, SW73 SW_Push, SW74 SW_Push, SW75 SW_Push, SW76 SW_Push, SW77 SW_Push, SW78 SW_Push, SW79 SW_Push, SW8 SW_Push, SW80 SW_Push, SW81 SW_Push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

Commit message: Last things Ill work on for PCB wise.
Parts:
- S2, S3, SW1, SW10, SW11, SW12, SW13, SW14, SW15, SW16, SW17, SW18, SW19, SW2, SW20, SW21, SW22, SW23, SW24, SW25, SW26, SW27, SW28, SW29, SW3, SW30, SW31, SW32, SW33, SW34, SW35, SW36, SW37, SW38, SW39, SW4, SW40, SW41, SW42, SW43, SW44, SW45, SW46, SW47, SW48, SW49, SW5, SW50, SW51, SW52, SW53, SW54, SW55, SW56, SW57, SW58, SW59, SW6, SW60, SW61, SW62, SW63, SW64, SW65, SW66, SW67, SW68, SW69, SW7, SW70, SW71, SW72, SW73, SW74, SW75, SW76, SW77, SW78, SW79, SW8, SW80, SW81, SW82, SW83, SW84, SW85, SW86, SW87, SW88, SW89, SW9, SW90, SW91, SW92, SW93, SW94, SW95, SW96, SW97: moved to B.Cu
- moved H12 40.4 mm to (449.2, 132.5)
- moved H11 20.3 mm to (395.3, 62.7)
- moved H7 9.95 mm to (43.7, 62.7)
- moved H10 7.98 mm to (331.8, 62.7)
- moved H8 7.94 mm to (138.9, 62.7)
- moved H9 7.94 mm to (235.7, 62.7)
- turned S2 to 180 degrees
- turned S3 to 180 degrees
- turned SW1 to 180 degrees
- turned SW10 to 180 degrees
- turned SW11 to 180 degrees
- turned SW12 to 180 degrees
- turned SW13 to 180 degrees
- turned SW14 to 180 degrees
- turned SW15 to 180 degrees
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Routing:
- net /COL9: track 1313.7 -> 985.4 mm, vias 0 -> 16
- net /COL1: track 521.2 -> 654.1 mm, vias 2 -> 12
- net /COL2: track 497.3 -> 629.0 mm, vias 2 -> 14
- net /COL0: track 533.7 -> 658.3 mm, vias 0 -> 4
- net /Row 1: track 491.4 -> 410.8 mm
- net /COL3: track 497.8 -> 562.5 mm, vias 2 -> 14
- net /COL7: track 441.9 -> 488.9 mm, vias 3 -> 16
- net /COL5: track 509.9 -> 552.6 mm, vias 2 -> 16
- net /COL10: track 380.1 -> 416.6 mm, vias 1 -> 12
- net /COL16: track 267.6 -> 234.6 mm, vias 3 -> 16
- net /Fn Row: track 408.8 -> 381.2 mm
- net /COL17: track 237.6 -> 210.2 mm, vias 3 -> 10
- net /COL15: track 281.0 -> 256.6 mm, vias 3 -> 12
- net /COL6: track 489.5 -> 512.2 mm, vias 4 -> 16
- net /COL4: track 538.8 -> 558.9 mm, vias 2 -> 14
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- added copper zone on F.Cu, net Net-(A1-GND-Pad13)
Other:
- board size 413.5 x 159.5 mm -> 413.5 x 148.4 mm
- board text added: "#KITSU"
- board text added: "@Wolfentech"
- board text added: "Ahrigato"
- board text added: "Videsh Arivazhagan"
