File: PCB FILES/vBoard/vBoard.kicad_sch (KiCad schematic)
At the start: 2 parts, among them SW1 SW_Push

Commit message: ill journal tomorrow
Parts:
- added D1, D10, D11, D12, D13, D14, D15, D16, D18, D19, D2, D20, D21, D22, D23, D24, D25, D26, D27, D28, D29, D3, D30, D31, D32, D33, D34, D35, D36, D37, D38, D39, D4, D40, D41, D42, D43, D44, D45, D46, D47, D48, D49, D5, D50, D51, D52, D53, D54, D55, D56, D57, D58, D59, D6, D60, D61, D62, D63, D64, D65, D66, D67, D68, D69, D7, D70, D71, D72, D73, D74, D75, D76, D77, D78, D79, D8, D80, D81, D82, D83, D84, D85, D86, D87, D88, D89, D9, D90, D91, D92, D93, D94, D95, D96, D97, D98: 1N4148, Diode_THT:D_DO-35_SOD27_P7.62mm_Horizontal, symbol Diode:1N4148
- added S1, S10, S11, S12, S2, S3, S4, S5, S6, S7, S8, S9: MX_stab, PCM_marbastlib-mx:STAB_MX_P_6.25u, symbol PCM_marbastlib-mx:MX_stab
- added SW10, SW11, SW12, SW13, SW14, SW15, SW16, SW18, SW19, SW2, SW20, SW21, SW22, SW23, SW24, SW25, SW26, SW27, SW28, SW29, SW3, SW30, SW31, SW32, SW33, SW34, SW35, SW36, SW37, SW38, SW39, SW4, SW40, SW41, SW42, SW43, SW44, SW45, SW46, SW47, SW48, SW49, SW5, SW50, SW51, SW52, SW53, SW54, SW55, SW56, SW57, SW58, SW59, SW6, SW60, SW61, SW62, SW63, SW64, SW65, SW66, SW67, SW68, SW69, SW7, SW70, SW71, SW72, SW73, SW74, SW75, SW76, SW77, SW78, SW79, SW8, SW80, SW81, SW82, SW83, SW84, SW85, SW86, SW87, SW88, SW89, SW9, SW90, SW91, SW92, SW93, SW94, SW95, SW96, SW97, SW98: SW_Push, Button_Switch_THT:SW_NKK_GW12LJP, symbol Switch:SW_Push
Connections:
- net COL0: now reaches SW1.1
- net COL0: now also SW18.1, SW36.1, SW54.1, SW70.1, SW86.1
- net at SW1.2: now also D1.2 (A)
- new net: D44.2 (A), SW44.2
- new net: D34.2 (A), SW34.2
- new net: D5.2 (A), SW5.2
- new net: D48.2 (A), SW48.2
- new net: D89.2 (A), SW89.2
- new net: D31.2 (A), SW31.2
- new net: D40.2 (A), SW40.2
- new net: D92.2 (A), SW92.2
- new net: D79.2 (A), SW79.2
- new net: D36.2 (A), SW36.2
- new net: D60.2 (A), SW60.2
- new net: D22.2 (A), SW22.2
- new net: D49.2 (A), SW49.2
- new net: D74.2 (A), SW74.2
- new net: D91.2 (A), SW91.2
- new net: D72.2 (A), SW72.2
- new net: D16.2 (A), SW16.2
- new net: D98.2 (A), SW98.2
- new net: D21.2 (A), SW21.2
- new net: D80.2 (A), SW80.2
- new net: D95.2 (A), SW95.2
- new net: D30.2 (A), SW30.2
- new net: D28.2 (A), SW28.2
- new net: D24.2 (A), SW24.2
- new net: D65.2 (A), SW65.2
- new net: D43.2 (A), SW43.2
- new net: D11.2 (A), SW11.2
- new net: D25.2 (A), SW25.2
- new net: D63.2 (A), SW63.2
- new net: D85.2 (A), SW85.2
- new net: D10.2 (A), SW10.2
- new net: D4.2 (A), SW4.2
- new net: D8.2 (A), SW8.2
- new net: D68.2 (A), SW68.2
- new net: D55.2 (A), SW55.2
- new net: D61.2 (A), SW61.2
- new net: D23.2 (A), SW23.2
- new net: D29.2 (A), SW29.2
- new net: D35.2 (A), SW35.2
- new net: D39.2 (A), SW39.2
- new net: D67.2 (A), SW67.2
- new net: D96.2 (A), SW96.2
- new net: D38.2 (A), SW38.2
- new net: D81.2 (A), SW81.2
- new net: D77.2 (A), SW77.2
- new net: D73.2 (A), SW73.2
- new net: D6.2 (A), SW6.2
- new net: D9.2 (A), SW9.2
- new net: D86.2 (A), SW86.2
- new net: D87.2 (A), SW87.2
- new net: D47.2 (A), SW47.2
- new net: D52.2 (A), SW52.2
- new net: D14.2 (A), SW14.2
- new net: D64.2 (A), SW64.2
- new net: D46.2 (A), SW46.2
- new net: D57.2 (A), SW57.2
- new net: D37.2 (A), SW37.2
- new net: D78.2 (A), SW78.2
- new net: D27.2 (A), SW27.2
- new net: D71.2 (A), SW71.2
- new net: D69.2 (A), SW69.2
- new net: D82.2 (A), SW82.2
- new net: D90.2 (A), SW90.2
- new net: D20.2 (A), SW20.2
- new net: D19.2 (A), SW19.2
- new net: D54.2 (A), SW54.2
- new net: D26.2 (A), SW26.2
- new net: D56.2 (A), SW56.2
- new net: D7.2 (A), SW7.2
- new net: D70.2 (A), SW70.2
- new net: D66.2 (A), SW66.2
- new net: D84.2 (A), SW84.2
- new net: D58.2 (A), SW58.2
- new net: D2.2 (A), SW2.2
- new net: D33.2 (A), SW33.2
- new net: D59.2 (A), SW59.2
- new net: D45.2 (A), SW45.2
- new net: D75.2 (A), SW75.2
- new net: D18.2 (A), SW18.2
- new net: D42.2 (A), SW42.2
- new net: D93.2 (A), SW93.2
- new net: D53.2 (A), SW53.2
- new net: D76.2 (A), SW76.2
- new net: D51.2 (A), SW51.2
- new net: D3.2 (A), SW3.2
- new net: D32.2 (A), SW32.2
- new net: D83.2 (A), SW83.2
- new net: D50.2 (A), SW50.2
- new net: D62.2 (A), SW62.2
- new net: D12.2 (A), SW12.2
- new net: D97.2 (A), SW97.2
- new net: D41.2 (A), SW41.2
- new net: D88.2 (A), SW88.2
- new net: D94.2 (A), SW94.2
- new net: D13.2 (A), SW13.2
- new net: D15.2 (A), SW15.2
- new net COL1: SW19.1, SW2.1, SW37.1, SW55.1, SW71.1, SW87.1
- new net COL10: SW11.1, SW28.1, SW46.1, SW64.1, SW80.1, SW92.1
- new net COL11: SW12.1, SW29.1, SW47.1, SW65.1, SW81.1
- new net COL12: D54.1 (K), D55.1 (K), D56.1 (K), D57.1 (K), D58.1 (K), D59.1 (K), D60.1 (K), D61.1 (K), D62.1 (K), D63.1 (K), D64.1 (K), D65.1 (K), D66.1 (K), D67.1 (K), D68.1 (K), D69.1 (K), SW13.1, SW30.1, SW48.1, SW66.1, SW96.1
- new net COL13: SW31.1, SW49.1, SW93.1, SW97.1
- new net COL14: SW14.1, SW32.1, SW50.1, SW67.1, SW82.1, SW98.1
- new net COL15: SW15.1, SW33.1, SW51.1, SW68.1, SW83.1, SW94.1
- new net COL16: SW16.1, SW34.1, SW52.1, SW69.1, SW84.1, SW95.1
- new net COL17: SW35.1, SW53.1, SW85.1
- new net COL2: SW20.1, SW3.1, SW38.1, SW56.1, SW72.1, SW88.1
- new net COL3: SW21.1, SW39.1, SW4.1, SW57.1, SW73.1
- new net COL4: SW22.1, SW40.1, SW5.1, SW58.1, SW74.1
- new net COL5: SW23.1, SW41.1, SW59.1, SW6.1, SW75.1, SW89.1
- new net COL6: SW24.1, SW42.1, SW60.1, SW7.1, SW76.1
- new net COL7: SW25.1, SW43.1, SW61.1, SW77.1, SW8.1
- new net COL8: SW26.1, SW44.1, SW62.1, SW78.1, SW9.1, SW90.1
- new net COL9: SW10.1, SW27.1, SW45.1, SW63.1, SW79.1, SW91.1
- new net Fn Row: D1.1 (K), D10.1 (K), D11.1 (K), D12.1 (K), D13.1 (K), D14.1 (K), D15.1 (K), D16.1 (K), D2.1 (K), D3.1 (K), D4.1 (K), D5.1 (K), D6.1 (K), D7.1 (K), D8.1 (K), D9.1 (K)
- new net Row 1: D18.1 (K), D19.1 (K), D20.1 (K), D21.1 (K), D22.1 (K), D23.1 (K), D24.1 (K), D25.1 (K), D26.1 (K), D27.1 (K), D28.1 (K), D29.1 (K), D30.1 (K), D31.1 (K), D32.1 (K), D33.1 (K), D34.1 (K), D35.1 (K)
- new net Row 2: D36.1 (K), D37.1 (K), D38.1 (K), D39.1 (K), D40.1 (K), D41.1 (K), D42.1 (K), D43.1 (K), D44.1 (K), D45.1 (K), D46.1 (K), D47.1 (K), D48.1 (K), D49.1 (K), D50.1 (K), D51.1 (K), D52.1 (K), D53.1 (K)
- new net Row 4: D70.1 (K), D71.1 (K), D72.1 (K), D73.1 (K), D74.1 (K), D75.1 (K), D76.1 (K), D77.1 (K), D78.1 (K), D79.1 (K), D80.1 (K), D81.1 (K), D82.1 (K), D83.1 (K), D84.1 (K), D85.1 (K), D93.1 (K)
- new net Row 5: D86.1 (K), D87.1 (K), D88.1 (K), D89.1 (K), D90.1 (K), D91.1 (K), D92.1 (K), D94.1 (K), D95.1 (K), D96.1 (K), D97.1 (K), D98.1 (K)
Other:
- moved on the sheet: A1, SW1

Commit message: Finally updated logs
Parts:
- removed S1, S10, S11, S12, S3, S4, S5, S6, S7, S8, S9: MX_stab, PCM_marbastlib-mx:STAB_MX_P_6.25u, symbol PCM_marbastlib-mx:MX_stab
- added D98: 1N4148, Diode_SMD:D_SOD-123, symbol Diode:1N4148
- added SW98: RotaryEncoder_Switch, Rotary_Encoder:RotaryEncoder_Alps_EC11E-Switch_Vertical_H20mm, symbol Device:RotaryEncoder_Switch
- A1: footprint Module:RaspberryPi_Pico_Common_Unspecified -> Module:RaspberryPi_Pico_Common_THT
- D1, D10, D11, D12, D13, D14, D15, D16, D2, D3, D4, D5, D6, D7, D8, D9: footprint Diode_THT:D_DO-35_SOD27_P7.62mm_Horizontal -> Diode_SMD:D_SOD-123
- D17: renamed from D18; footprint Diode_THT:D_DO-35_SOD27_P7.62mm_Horizontal -> Diode_SMD:D_SOD-123
- D18: renamed from D19; footprint Diode_THT:D_DO-35_SOD27_P7.62mm_Horizontal -> Diode_SMD:D_SOD-123
- D19: renamed from D20; footprint Diode_THT:D_DO-35_SOD27_P7.62mm_Horizontal -> Diode_SMD:D_SOD-123
- D20: renamed from D21; footprint Diode_THT:D_DO-35_SOD27_P7.62mm_Horizontal -> Diode_SMD:D_SOD-123
- D21: renamed from D22; footprint Diode_THT:D_DO-35_SOD27_P7.62mm_Horizontal -> Diode_SMD:D_SOD-123
- D22: renamed from D23; footprint Diode_THT:D_DO-35_SOD27_P7.62mm_Horizontal -> Diode_SMD:D_SOD-123
- D23: renamed from D24; footprint Diode_THT:D_DO-35_SOD27_P7.62mm_Horizontal -> Diode_SMD:D_SOD-123
- D24: renamed from D25; footprint Diode_THT:D_DO-35_SOD27_P7.62mm_Horizontal -> Diode_SMD:D_SOD-123
- D25: renamed from D26; footprint Diode_THT:D_DO-35_SOD27_P7.62mm_Horizontal -> Diode_SMD:D_SOD-123
- D26: renamed from D27; footprint Diode_THT:D_DO-35_SOD27_P7.62mm_Horizontal -> Diode_SMD:D_SOD-123
- D27: renamed from D28; footprint Diode_THT:D_DO-35_SOD27_P7.62mm_Horizontal -> Diode_SMD:D_SOD-123
- D28: renamed from D29; footprint Diode_THT:D_DO-35_SOD27_P7.62mm_Horizontal -> Diode_SMD:D_SOD-123
- D29: renamed from D30; footprint Diode_THT:D_DO-35_SOD27_P7.62mm_Horizontal -> Diode_SMD:D_SOD-123
- D30: renamed from D31; footprint Diode_THT:D_DO-35_SOD27_P7.62mm_Horizontal -> Diode_SMD:D_SOD-123
- D31: renamed from D32; footprint Diode_THT:D_DO-35_SOD27_P7.62mm_Horizontal -> Diode_SMD:D_SOD-123
- D32: renamed from D33; footprint Diode_THT:D_DO-35_SOD27_P7.62mm_Horizontal -> Diode_SMD:D_SOD-123
- D33: renamed from D34; footprint Diode_THT:D_DO-35_SOD27_P7.62mm_Horizontal -> Diode_SMD:D_SOD-123
- D34: renamed from D35; footprint Diode_THT:D_DO-35_SOD27_P7.62mm_Horizontal -> Diode_SMD:D_SOD-123
- D35: renamed from D36; footprint Diode_THT:D_DO-35_SOD27_P7.62mm_Horizontal -> Diode_SMD:D_SOD-123
- D36: renamed from D37; footprint Diode_THT:D_DO-35_SOD27_P7.62mm_Horizontal -> Diode_SMD:D_SOD-123
- D37: renamed from D38; footprint Diode_THT:D_DO-35_SOD27_P7.62mm_Horizontal -> Diode_SMD:D_SOD-123
- D38: renamed from D39; footprint Diode_THT:D_DO-35_SOD27_P7.62mm_Horizontal -> Diode_SMD:D_SOD-123
- D39: renamed from D40; footprint Diode_THT:D_DO-35_SOD27_P7.62mm_Horizontal -> Diode_SMD:D_SOD-123
- D40: renamed from D41; footprint Diode_THT:D_DO-35_SOD27_P7.62mm_Horizontal -> Diode_SMD:D_SOD-123
- D41: renamed from D42; footprint Diode_THT:D_DO-35_SOD27_P7.62mm_Horizontal -> Diode_SMD:D_SOD-123
- D42: renamed from D43; footprint Diode_THT:D_DO-35_SOD27_P7.62mm_Horizontal -> Diode_SMD:D_SOD-123
- D43: renamed from D44; footprint Diode_THT:D_DO-35_SOD27_P7.62mm_Horizontal -> Diode_SMD:D_SOD-123
- D44: renamed from D45; footprint Diode_THT:D_DO-35_SOD27_P7.62mm_Horizontal -> Diode_SMD:D_SOD-123
- D45: renamed from D46; footprint Diode_THT:D_DO-35_SOD27_P7.62mm_Horizontal -> Diode_SMD:D_SOD-123
- D46: renamed from D47; footprint Diode_THT:D_DO-35_SOD27_P7.62mm_Horizontal -> Diode_SMD:D_SOD-123
- D47: renamed from D48; footprint Diode_THT:D_DO-35_SOD27_P7.62mm_Horizontal -> Diode_SMD:D_SOD-123
- D48: renamed from D49; footprint Diode_THT:D_DO-35_SOD27_P7.62mm_Horizontal -> Diode_SMD:D_SOD-123
- D49: renamed from D50; footprint Diode_THT:D_DO-35_SOD27_P7.62mm_Horizontal -> Diode_SMD:D_SOD-123
- D50: renamed from D51; footprint Diode_THT:D_DO-35_SOD27_P7.62mm_Horizontal -> Diode_SMD:D_SOD-123
- D51: renamed from D52; footprint Diode_THT:D_DO-35_SOD27_P7.62mm_Horizontal -> Diode_SMD:D_SOD-123
- D52: renamed from D53; footprint Diode_THT:D_DO-35_SOD27_P7.62mm_Horizontal -> Diode_SMD:D_SOD-123
- D53: renamed from D54; footprint Diode_THT:D_DO-35_SOD27_P7.62mm_Horizontal -> Diode_SMD:D_SOD-123
- D54: renamed from D55; footprint Diode_THT:D_DO-35_SOD27_P7.62mm_Horizontal -> Diode_SMD:D_SOD-123
- D55: renamed from D56; footprint Diode_THT:D_DO-35_SOD27_P7.62mm_Horizontal -> Diode_SMD:D_SOD-123
- D56: renamed from D57; footprint Diode_THT:D_DO-35_SOD27_P7.62mm_Horizontal -> Diode_SMD:D_SOD-123
- D57: renamed from D58; footprint Diode_THT:D_DO-35_SOD27_P7.62mm_Horizontal -> Diode_SMD:D_SOD-123
- D58: renamed from D59; footprint Diode_THT:D_DO-35_SOD27_P7.62mm_Horizontal -> Diode_SMD:D_SOD-123
- D59: renamed from D60; footprint Diode_THT:D_DO-35_SOD27_P7.62mm_Horizontal -> Diode_SMD:D_SOD-123
- D60: renamed from D61; footprint Diode_THT:D_DO-35_SOD27_P7.62mm_Horizontal -> Diode_SMD:D_SOD-123
- D61: renamed from D62; footprint Diode_THT:D_DO-35_SOD27_P7.62mm_Horizontal -> Diode_SMD:D_SOD-123
- D62: renamed from D63; footprint Diode_THT:D_DO-35_SOD27_P7.62mm_Horizontal -> Diode_SMD:D_SOD-123
- D63: renamed from D64; footprint Diode_THT:D_DO-35_SOD27_P7.62mm_Horizontal -> Diode_SMD:D_SOD-123
- D64: renamed from D65; footprint Diode_THT:D_DO-35_SOD27_P7.62mm_Horizontal -> Diode_SMD:D_SOD-123
- D65: renamed from D66; footprint Diode_THT:D_DO-35_SOD27_P7.62mm_Horizontal -> Diode_SMD:D_SOD-123
- D66: renamed from D67; footprint Diode_THT:D_DO-35_SOD27_P7.62mm_Horizontal -> Diode_SMD:D_SOD-123
- D67: renamed from D68; footprint Diode_THT:D_DO-35_SOD27_P7.62mm_Horizontal -> Diode_SMD:D_SOD-123
- D68: renamed from D69; footprint Diode_THT:D_DO-35_SOD27_P7.62mm_Horizontal -> Diode_SMD:D_SOD-123
- D69: renamed from D70; footprint Diode_THT:D_DO-35_SOD27_P7.62mm_Horizontal -> Diode_SMD:D_SOD-123
- D70: renamed from D71; footprint Diode_THT:D_DO-35_SOD27_P7.62mm_Horizontal -> Diode_SMD:D_SOD-123
- D71: renamed from D72; footprint Diode_THT:D_DO-35_SOD27_P7.62mm_Horizontal -> Diode_SMD:D_SOD-123
- D72: renamed from D73; footprint Diode_THT:D_DO-35_SOD27_P7.62mm_Horizontal -> Diode_SMD:D_SOD-123
- D73: renamed from D74; footprint Diode_THT:D_DO-35_SOD27_P7.62mm_Horizontal -> Diode_SMD:D_SOD-123
- D74: renamed from D75; footprint Diode_THT:D_DO-35_SOD27_P7.62mm_Horizontal -> Diode_SMD:D_SOD-123
- D75: renamed from D76; footprint Diode_THT:D_DO-35_SOD27_P7.62mm_Horizontal -> Diode_SMD:D_SOD-123
- D76: renamed from D77; footprint Diode_THT:D_DO-35_SOD27_P7.62mm_Horizontal -> Diode_SMD:D_SOD-123
- D77: renamed from D78; footprint Diode_THT:D_DO-35_SOD27_P7.62mm_Horizontal -> Diode_SMD:D_SOD-123
- D78: renamed from D79; footprint Diode_THT:D_DO-35_SOD27_P7.62mm_Horizontal -> Diode_SMD:D_SOD-123
- D79: renamed from D80; footprint Diode_THT:D_DO-35_SOD27_P7.62mm_Horizontal -> Diode_SMD:D_SOD-123
- D80: renamed from D81; footprint Diode_THT:D_DO-35_SOD27_P7.62mm_Horizontal -> Diode_SMD:D_SOD-123
- D81: renamed from D82; footprint Diode_THT:D_DO-35_SOD27_P7.62mm_Horizontal -> Diode_SMD:D_SOD-123
- D82: renamed from D83; footprint Diode_THT:D_DO-35_SOD27_P7.62mm_Horizontal -> Diode_SMD:D_SOD-123
- D83: renamed from D84; footprint Diode_THT:D_DO-35_SOD27_P7.62mm_Horizontal -> Diode_SMD:D_SOD-123
- D84: renamed from D85; footprint Diode_THT:D_DO-35_SOD27_P7.62mm_Horizontal -> Diode_SMD:D_SOD-123
- D85: renamed from D86; footprint Diode_THT:D_DO-35_SOD27_P7.62mm_Horizontal -> Diode_SMD:D_SOD-123
- D86: renamed from D87; footprint Diode_THT:D_DO-35_SOD27_P7.62mm_Horizontal -> Diode_SMD:D_SOD-123
- D87: renamed from D88; footprint Diode_THT:D_DO-35_SOD27_P7.62mm_Horizontal -> Diode_SMD:D_SOD-123
- D88: renamed from D89; footprint Diode_THT:D_DO-35_SOD27_P7.62mm_Horizontal -> Diode_SMD:D_SOD-123
- D89: renamed from D90; footprint Diode_THT:D_DO-35_SOD27_P7.62mm_Horizontal -> Diode_SMD:D_SOD-123
- D90: renamed from D91; footprint Diode_THT:D_DO-35_SOD27_P7.62mm_Horizontal -> Diode_SMD:D_SOD-123
- D91: renamed from D92; footprint Diode_THT:D_DO-35_SOD27_P7.62mm_Horizontal -> Diode_SMD:D_SOD-123
- D92: renamed from D93; footprint Diode_THT:D_DO-35_SOD27_P7.62mm_Horizontal -> Diode_SMD:D_SOD-123
- D93: renamed from D94; footprint Diode_THT:D_DO-35_SOD27_P7.62mm_Horizontal -> Diode_SMD:D_SOD-123
- D94: renamed from D95; footprint Diode_THT:D_DO-35_SOD27_P7.62mm_Horizontal -> Diode_SMD:D_SOD-123
- D95: renamed from D96; footprint Diode_THT:D_DO-35_SOD27_P7.62mm_Horizontal -> Diode_SMD:D_SOD-123
- D96: renamed from D97; footprint Diode_THT:D_DO-35_SOD27_P7.62mm_Horizontal -> Diode_SMD:D_SOD-123
- D97: renamed from D98; footprint Diode_THT:D_DO-35_SOD27_P7.62mm_Horizontal -> Diode_SMD:D_SOD-123
- S9: renamed from S2; footprint PCM_marbastlib-mx:STAB_MX_P_6.25u -> PCM_marbastlib-mx:STAB_MX_P_2u
- SW1, SW10, SW11, SW12, SW13, SW14, SW15, SW16, SW2, SW3, SW4, SW5, SW6, SW7, SW8, SW9: footprint Button_Switch_THT:SW_NKK_GW12LJP -> PCM_marbastlib-mx:SW_MX_HS_CPG151101S11_1u
- SW17: renamed from SW18; footprint Button_Switch_THT:SW_NKK_GW12LJP -> PCM_marbastlib-mx:SW_MX_HS_CPG151101S11_1u
- SW18: renamed from SW19; footprint Button_Switch_THT:SW_NKK_GW12LJP -> PCM_marbastlib-mx:SW_MX_HS_CPG151101S11_1u
- SW19: renamed from SW20; footprint Button_Switch_THT:SW_NKK_GW12LJP -> PCM_marbastlib-mx:SW_MX_HS_CPG151101S11_1u
- SW20: renamed from SW21; footprint Button_Switch_THT:SW_NKK_GW12LJP -> PCM_marbastlib-mx:SW_MX_HS_CPG151101S11_1u
- SW21: renamed from SW22; footprint Button_Switch_THT:SW_NKK_GW12LJP -> PCM_marbastlib-mx:SW_MX_HS_CPG151101S11_1u
- SW22: renamed from SW23; footprint Button_Switch_THT:SW_NKK_GW12LJP -> PCM_marbastlib-mx:SW_MX_HS_CPG151101S11_1u
- SW23: renamed from SW24; footprint Button_Switch_THT:SW_NKK_GW12LJP -> PCM_marbastlib-mx:SW_MX_HS_CPG151101S11_1u
- SW24: renamed from SW25; footprint Button_Switch_THT:SW_NKK_GW12LJP -> PCM_marbastlib-mx:SW_MX_HS_CPG151101S11_1u
- SW25: renamed from SW26; footprint Button_Switch_THT:SW_NKK_GW12LJP -> PCM_marbastlib-mx:SW_MX_HS_CPG151101S11_1u
- SW26: renamed from SW27; footprint Button_Switch_THT:SW_NKK_GW12LJP -> PCM_marbastlib-mx:SW_MX_HS_CPG151101S11_1u
- SW27: renamed from SW28; footprint Button_Switch_THT:SW_NKK_GW12LJP -> PCM_marbastlib-mx:SW_MX_HS_CPG151101S11_1u
- SW28: renamed from SW29; footprint Button_Switch_THT:SW_NKK_GW12LJP -> PCM_marbastlib-mx:SW_MX_HS_CPG151101S11_1u
- SW29: renamed from SW30; footprint Button_Switch_THT:SW_NKK_GW12LJP -> PCM_marbastlib-mx:SW_MX_HS_CPG151101S11_1u
- SW30: renamed from SW31; footprint Button_Switch_THT:SW_NKK_GW12LJP -> PCM_marbastlib-mx:SW_MX_HS_CPG151101S11_1u
- SW31: renamed from SW32; footprint Button_Switch_THT:SW_NKK_GW12LJP -> PCM_marbastlib-mx:SW_MX_HS_CPG151101S11_1u
- SW32: renamed from SW33; footprint Button_Switch_THT:SW_NKK_GW12LJP -> PCM_marbastlib-mx:SW_MX_HS_CPG151101S11_1u
- SW33: renamed from SW34; footprint Button_Switch_THT:SW_NKK_GW12LJP -> PCM_marbastlib-mx:SW_MX_HS_CPG151101S11_1u
- SW34: renamed from SW35; footprint Button_Switch_THT:SW_NKK_GW12LJP -> PCM_marbastlib-mx:SW_MX_HS_CPG151101S11_1u
- SW35: renamed from SW36; footprint Button_Switch_THT:SW_NKK_GW12LJP -> PCM_marbastlib-mx:SW_MX_HS_CPG151101S11_1u
- SW36: renamed from SW37; footprint Button_Switch_THT:SW_NKK_GW12LJP -> PCM_marbastlib-mx:SW_MX_HS_CPG151101S11_1u
- SW37: renamed from SW38; footprint Button_Switch_THT:SW_NKK_GW12LJP -> PCM_marbastlib-mx:SW_MX_HS_CPG151101S11_1u
- SW38: renamed from SW39; footprint Button_Switch_THT:SW_NKK_GW12LJP -> PCM_marbastlib-mx:SW_MX_HS_CPG151101S11_1u
- SW39: renamed from SW40; footprint Button_Switch_THT:SW_NKK_GW12LJP -> PCM_marbastlib-mx:SW_MX_HS_CPG151101S11_1u
- SW40: renamed from SW41; footprint Button_Switch_THT:SW_NKK_GW12LJP -> PCM_marbastlib-mx:SW_MX_HS_CPG151101S11_1u
- SW41: renamed from SW42; footprint Button_Switch_THT:SW_NKK_GW12LJP -> PCM_marbastlib-mx:SW_MX_HS_CPG151101S11_1u
- SW42: renamed from SW43; footprint Button_Switch_THT:SW_NKK_GW12LJP -> PCM_marbastlib-mx:SW_MX_HS_CPG151101S11_1u
- SW43: renamed from SW44; footprint Button_Switch_THT:SW_NKK_GW12LJP -> PCM_marbastlib-mx:SW_MX_HS_CPG151101S11_1u
- SW44: renamed from SW45; footprint Button_Switch_THT:SW_NKK_GW12LJP -> PCM_marbastlib-mx:SW_MX_HS_CPG151101S11_1u
- SW45: renamed from SW46; footprint Button_Switch_THT:SW_NKK_GW12LJP -> PCM_marbastlib-mx:SW_MX_HS_CPG151101S11_1u
- SW46: renamed from SW47; footprint Button_Switch_THT:SW_NKK_GW12LJP -> PCM_marbastlib-mx:SW_MX_HS_CPG151101S11_1u
- SW47: renamed from SW48; footprint Button_Switch_THT:SW_NKK_GW12LJP -> PCM_marbastlib-mx:SW_MX_HS_CPG151101S11_1u
- SW48: renamed from SW49; footprint Button_Switch_THT:SW_NKK_GW12LJP -> PCM_marbastlib-mx:SW_MX_HS_CPG151101S11_1u
- SW49: renamed from SW50; footprint Button_Switch_THT:SW_NKK_GW12LJP -> PCM_marbastlib-mx:SW_MX_HS_CPG151101S11_1u
- SW50: renamed from SW51; footprint Button_Switch_THT:SW_NKK_GW12LJP -> PCM_marbastlib-mx:SW_MX_HS_CPG151101S11_1u
- SW51: renamed from SW52; footprint Button_Switch_THT:SW_NKK_GW12LJP -> PCM_marbastlib-mx:SW_MX_HS_CPG151101S11_1u
- SW52: renamed from SW53; footprint Button_Switch_THT:SW_NKK_GW12LJP -> PCM_marbastlib-mx:SW_MX_HS_CPG151101S11_1u
- SW53: renamed from SW54; footprint Button_Switch_THT:SW_NKK_GW12LJP -> PCM_marbastlib-mx:SW_MX_HS_CPG151101S11_1u
- SW54: renamed from SW55; footprint Button_Switch_THT:SW_NKK_GW12LJP -> PCM_marbastlib-mx:SW_MX_HS_CPG151101S11_1u
- SW55: renamed from SW56; footprint Button_Switch_THT:SW_NKK_GW12LJP -> PCM_marbastlib-mx:SW_MX_HS_CPG151101S11_1u
- SW56: renamed from SW57; footprint Button_Switch_THT:SW_NKK_GW12LJP -> PCM_marbastlib-mx:SW_MX_HS_CPG151101S11_1u
- SW57: renamed from SW58; footprint Button_Switch_THT:SW_NKK_GW12LJP -> PCM_marbastlib-mx:SW_MX_HS_CPG151101S11_1u
- SW58: renamed from SW59; footprint Button_Switch_THT:SW_NKK_GW12LJP -> PCM_marbastlib-mx:SW_MX_HS_CPG151101S11_1u
- SW59: renamed from SW60; footprint Button_Switch_THT:SW_NKK_GW12LJP -> PCM_marbastlib-mx:SW_MX_HS_CPG151101S11_1u
- SW60: renamed from SW61; footprint Button_Switch_THT:SW_NKK_GW12LJP -> PCM_marbastlib-mx:SW_MX_HS_CPG151101S11_1u
- SW61: renamed from SW62; footprint Button_Switch_THT:SW_NKK_GW12LJP -> PCM_marbastlib-mx:SW_MX_HS_CPG151101S11_1u
- SW62: renamed from SW63; footprint Button_Switch_THT:SW_NKK_GW12LJP -> PCM_marbastlib-mx:SW_MX_HS_CPG151101S11_1u
- SW63: renamed from SW64; footprint Button_Switch_THT:SW_NKK_GW12LJP -> PCM_marbastlib-mx:SW_MX_HS_CPG151101S11_1u
- SW64: renamed from SW65; footprint Button_Switch_THT:SW_NKK_GW12LJP -> PCM_marbastlib-mx:SW_MX_HS_CPG151101S11_1u
- SW65: renamed from SW66; footprint Button_Switch_THT:SW_NKK_GW12LJP -> PCM_marbastlib-mx:SW_MX_HS_CPG151101S11_1u
- SW66: renamed from SW67; footprint Button_Switch_THT:SW_NKK_GW12LJP -> PCM_marbastlib-mx:SW_MX_HS_CPG151101S11_1u
- SW67: renamed from SW68; footprint Button_Switch_THT:SW_NKK_GW12LJP -> PCM_marbastlib-mx:SW_MX_HS_CPG151101S11_1u
- SW68: renamed from SW69; footprint Button_Switch_THT:SW_NKK_GW12LJP -> PCM_marbastlib-mx:SW_MX_HS_CPG151101S11_1u
- SW69: renamed from SW70; footprint Button_Switch_THT:SW_NKK_GW12LJP -> PCM_marbastlib-mx:SW_MX_HS_CPG151101S11_1u
- SW70: renamed from SW71; footprint Button_Switch_THT:SW_NKK_GW12LJP -> PCM_marbastlib-mx:SW_MX_HS_CPG151101S11_1u
- SW71: renamed from SW72; footprint Button_Switch_THT:SW_NKK_GW12LJP -> PCM_marbastlib-mx:SW_MX_HS_CPG151101S11_1u
- SW72: renamed from SW73; footprint Button_Switch_THT:SW_NKK_GW12LJP -> PCM_marbastlib-mx:SW_MX_HS_CPG151101S11_1u
- SW73: renamed from SW74; footprint Button_Switch_THT:SW_NKK_GW12LJP -> PCM_marbastlib-mx:SW_MX_HS_CPG151101S11_1u
- SW74: renamed from SW75; footprint Button_Switch_THT:SW_NKK_GW12LJP -> PCM_marbastlib-mx:SW_MX_HS_CPG151101S11_1u
- SW75: renamed from SW76; footprint Button_Switch_THT:SW_NKK_GW12LJP -> PCM_marbastlib-mx:SW_MX_HS_CPG151101S11_1u
- SW76: renamed from SW77; footprint Button_Switch_THT:SW_NKK_GW12LJP -> PCM_marbastlib-mx:SW_MX_HS_CPG151101S11_1u
- SW77: renamed from SW78; footprint Button_Switch_THT:SW_NKK_GW12LJP -> PCM_marbastlib-mx:SW_MX_HS_CPG151101S11_1u
- SW78: renamed from SW79; footprint Button_Switch_THT:SW_NKK_GW12LJP -> PCM_marbastlib-mx:SW_MX_HS_CPG151101S11_1u
- SW79: renamed from SW80; footprint Button_Switch_THT:SW_NKK_GW12LJP -> PCM_marbastlib-mx:SW_MX_HS_CPG151101S11_1u
- SW80: renamed from SW81; footprint Button_Switch_THT:SW_NKK_GW12LJP -> PCM_marbastlib-mx:SW_MX_HS_CPG151101S11_1u
- SW81: renamed from SW82; footprint Button_Switch_THT:SW_NKK_GW12LJP -> PCM_marbastlib-mx:SW_MX_HS_CPG151101S11_1u
- SW82: renamed from SW83; footprint Button_Switch_THT:SW_NKK_GW12LJP -> PCM_marbastlib-mx:SW_MX_HS_CPG151101S11_1u
- SW83: renamed from SW84; footprint Button_Switch_THT:SW_NKK_GW12LJP -> PCM_marbastlib-mx:SW_MX_HS_CPG151101S11_1u
- SW84: renamed from SW85; footprint Button_Switch_THT:SW_NKK_GW12LJP -> PCM_marbastlib-mx:SW_MX_HS_CPG151101S11_1u
- SW85: renamed from SW86; footprint Button_Switch_THT:SW_NKK_GW12LJP -> PCM_marbastlib-mx:SW_MX_HS_CPG151101S11_1u
- SW86: renamed from SW87; footprint Button_Switch_THT:SW_NKK_GW12LJP -> PCM_marbastlib-mx:SW_MX_HS_CPG151101S11_1u
- SW87: renamed from SW88; footprint Button_Switch_THT:SW_NKK_GW12LJP -> PCM_marbastlib-mx:SW_MX_HS_CPG151101S11_1u
- SW88: renamed from SW89; footprint Button_Switch_THT:SW_NKK_GW12LJP -> PCM_marbastlib-mx:SW_MX_HS_CPG151101S11_1u
- SW89: renamed from SW90; footprint Button_Switch_THT:SW_NKK_GW12LJP -> PCM_marbastlib-mx:SW_MX_HS_CPG151101S11_1u
- SW90: renamed from SW91; footprint Button_Switch_THT:SW_NKK_GW12LJP -> PCM_marbastlib-mx:SW_MX_HS_CPG151101S11_1u
- SW91: renamed from SW92; footprint Button_Switch_THT:SW_NKK_GW12LJP -> PCM_marbastlib-mx:SW_MX_HS_CPG151101S11_1u
- SW92: renamed from SW93; footprint Button_Switch_THT:SW_NKK_GW12LJP -> PCM_marbastlib-mx:SW_MX_HS_CPG151101S11_1u
- SW93: renamed from SW94; footprint Button_Switch_THT:SW_NKK_GW12LJP -> PCM_marbastlib-mx:SW_MX_HS_CPG151101S11_1u
- SW94: renamed from SW95; footprint Button_Switch_THT:SW_NKK_GW12LJP -> PCM_marbastlib-mx:SW_MX_HS_CPG151101S11_1u
- SW95: renamed from SW96; footprint Button_Switch_THT:SW_NKK_GW12LJP -> PCM_marbastlib-mx:SW_MX_HS_CPG151101S11_1u
- SW96: renamed from SW97; footprint Button_Switch_THT:SW_NKK_GW12LJP -> PCM_marbastlib-mx:SW_MX_HS_CPG151101S11_1u
- SW97: renamed from SW98; footprint Button_Switch_THT:SW_NKK_GW12LJP -> PCM_marbastlib-mx:SW_MX_HS_CPG151101S11_1u
Connections:
- net COL0: now also A1.9 (GPIO6)
- net COL1: now also A1.10 (GPIO7)
- net COL10: now also A1.21 (GPIO16)
- net COL11: now also A1.22 (GPIO17)
- net COL12: now also A1.24 (GPIO18); no longer D53.1 (K), D54.1 (K), D55.1 (K), D56.1 (K), D57.1 (K), D58.1 (K), D59.1 (K), D60.1 (K), D61.1 (K), D62.1 (K), D63.1 (K), D64.1 (K), D65.1 (K), D66.1 (K), D67.1 (K), D68.1 (K)
- net COL13: now also A1.25 (GPIO19)
- net COL14: now also A1.26 (GPIO20)
- net COL15: now also A1.27 (GPIO21)
- net COL16: now also A1.29 (GPIO22)
- net COL17: now also A1.31 (GPIO26_ADC0), SW98.S1
- net COL2: now also A1.11 (GPIO8)
- net COL3: now also A1.12 (GPIO9)
- net COL4: now also A1.14 (GPIO10)
- net COL5: now also A1.15 (GPIO11)
- net COL6: now also A1.16 (GPIO12)
- net COL7: now also A1.17 (GPIO13)
- net COL8: now also A1.19 (GPIO14)
- net COL9: now also A1.20 (GPIO15)
- net Fn Row: now also A1.1 (GPIO0)
- net Row 1: now also A1.2 (GPIO1)
- net Row 2: now also A1.4 (GPIO2)
- net Row 4: now also A1.6 (GPIO4)
- net Row 5: now also A1.7 (GPIO5), D98.1 (K)
- net at A1.13 (GND), A1.18 (GND), A1.23 (GND)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: now also SW98.C
- net ROT0: now reaches A1.32 (GPIO27_ADC1)
- net ROT0: now also SW98.A
- net at A1.34 (GPIO28_ADC2): now also SW98.B
- net Row 3: now reaches A1.5 (GPIO3)
- net Row 3: now also D53.1 (K), D54.1 (K), D55.1 (K), D56.1 (K), D57.1 (K), D58.1 (K), D59.1 (K), D60.1 (K), D61.1 (K), D62.1 (K), D63.1 (K), D64.1 (K), D65.1 (K), D66.1 (K), D67.1 (K), D68.1 (K)
- new net: D98.2 (A), SW98.S2

Commit message: journaling kicad. Will work on cad after pcb.
Connections:
- net Row 5 is gone; now on net COL9: A1.7 (GPIO5), D85.1 (K), D86.1 (K), D87.1 (K), D88.1 (K), D89.1 (K), D90.1 (K), D91.1 (K), D93.1 (K), D94.1 (K), D95.1 (K), D96.1 (K), D97.1 (K), D98.1 (K)
Changed lines of the file:
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@@
 	(wire
 		(pts
+			(xy 332.74 124.46) (xy 313.69 124.46)
+		)
+		(stroke
+			(width 0)
+			(type default)
+		)
+	)
+	(wire
+		(pts
 			(xy 142.24 119.38) (xy 154.94 119.38)
 		)
@@
 	(wire
 		(pts
+			(xy 334.01 124.46) (xy 341.63 124.46)
+		)
+		(stroke
+			(width 0)
+			(type default)
+		)
+	)
+	(wire
+		(pts
 			(xy 394.97 228.6) (xy 394.97 119.38)
 		)
@@
 	(wire
 		(pts
+			(xy 330.2 99.06) (xy 341.63 99.06)
+		)
+		(stroke
+			(width 0)
+			(type default)
+		)
+	)
+	(wire
+		(pts
 			(xy 101.6 130.81) (xy 101.6 132.08)
 		)
@@
 	(wire
 		(pts
+			(xy 326.39 99.06) (xy 326.39 100.33)
+		)
+		(stroke
+			(width 0)
+			(type default)
+		)
+	)
+	(wire
+		(pts
 			(xy 53.34 40.64) (xy 53.34 54.61)
 		)
@@
 	(wire
 		(pts
+			(xy 326.39 100.33) (xy 334.01 100.33)
+		)
+		(stroke
+			(width 0)
+			(type default)
+		)
+	)
+	(wire
+		(pts
 			(xy 127 54.61) (xy 127 55.88)
 		)
@@
 	(wire
 		(pts
-			(xy 332.74 124.46) (xy 341.63 124.46)
-		)
-		(stroke
-			(width 0)
-			(type default)
-		)
-	)
-	(wire
-		(pts
 			(xy 53.34 29.21) (xy 53.34 39.37)
 		)
@@
 	(wire
 		(pts
+			(xy 313.69 97.79) (xy 330.2 97.79)
+		)
+		(stroke
+			(width 0)
+			(type default)
+		)
+	)
+	(wire
+		(pts
 			(xy 152.4 54.61) (xy 152.4 55.88)
 		)
@@
 	(wire
 		(pts
+			(xy 334.01 100.33) (xy 334.01 124.46)
+		)
+		(stroke
+			(width 0)
+			(type default)
+		)
+	)
+	(wire
+		(pts
 			(xy 288.29 152.4) (xy 304.8 152.4)
 		)
@@
 	(wire
 		(pts
+			(xy 313.69 124.46) (xy 313.69 97.79)
+		)
+		(stroke
+			(width 0)
+			(type default)
+		)
+	)
+	(wire
+		(pts
 			(xy 218.44 17.78) (xy 218.44 29.21)
 		)
@@
 	(wire
 		(pts
+			(xy 330.2 97.79) (xy 330.2 99.06)
+		)
+		(stroke
+			(width 0)
+			(type default)
+		)
+	)
+	(wire
+		(pts
 			(xy 27.94 80.01) (xy 27.94 105.41)
 		)
@@
 	(wire
 		(pts
+			(xy 320.04 99.06) (xy 326.39 99.06)
+		)
+		(stroke
+			(width 0)
+			(type default)
+		)
+	)
+	(wire
+		(pts
 			(xy 78.74 54.61) (xy 78.74 80.01)
 		)
@@
 	(wire
 		(pts
-			(xy 320.04 99.06) (xy 341.63 99.06)
-		)
-		(stroke
-			(width 0)
-			(type default)
-		)
-	)
-	(wire
-		(pts
 			(xy 180.34 53.34) (xy 180.34 54.61)
 		)
@@
 		)
 	)
-	(label "Row 5"
+	(label "COL9"
 		(at 332.74 99.06 0)
 		(effects
@@
 		)
 	)
-	(label "COL9"
+	(label "Row 5"
 		(at 332.74 124.46 0)
 		(effects

Commit message: Journaling and got some more work done.
Parts:
- removed S9: MX_stab, PCM_marbastlib-mx:STAB_MX_P_2u, symbol PCM_marbastlib-mx:MX_stab
- added H1, H10, H11, H12, H2, H3, H4, H5, H6, H7, H8, H9: MountingHole, MountingHole:MountingHole_3.2mm_M3, symbol Mechanical:MountingHole

Commit message: DRC fixes.
Changed lines of the file:
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@@
+		)
+	)
+	(label "COL9"
+		(at 332.74 99.06 0)
+		(effects
+			(font
+				(size 1.27 1.27)
+			)
+			(justify left bottom)
 		)
 	)
@@
 		)
 	)
+	(label "COL12"
+		(at 218.44 17.78 0)
+		(effects
+			(font
+				(size 1.27 1.27)
+			)
+			(justify left bottom)
+		)
+	)
+	(label "Row 5"
+		(at 12.7 165.1 0)
+		(effects
+			(font
+				(size 1.27 1.27)
+			)
+			(justify left bottom)
+		)
+	)
+	(label "COL14"
+		(at 243.84 17.78 0)
+		(effects
+			(font
+				(size 1.27 1.27)
+			)
+			(justify left bottom)
+		)
+	)
+	(label "Fn Row"
+		(at 332.74 86.36 0)
+		(effects
+			(font
+				(size 1.27 1.27)
+			)
+			(justify left bottom)
+		)
+	)
+	(label "COL5"
+		(at 332.74 114.3 0)
+		(effects
+			(font
+				(size 1.27 1.27)
+			)
+			(justify left bottom)
+		)
+	)
+	(label "COL11"
+		(at 392.43 91.44 0)
+		(effects
+			(font
+				(size 1.27 1.27)
+			)
+			(justify left bottom)
+		)
+	)
+	(label "COL10"
+		(at 193.04 17.78 0)
+		(effects
+			(font
+				(size 1.27 1.27)
+			)
+			(justify left bottom)
+		)
+	)
+	(label "COL13"
+		(at 392.43 96.52 0)
+		(effects
+			(font
+				(size 1.27 1.27)
+			)
+			(justify left bottom)
+		)
+	)
+	(label "COL12"
+		(at 392.43 93.98 0)
+		(effects
+			(font
+				(size 1.27 1.27)
+			)
+			(justify left bottom)
+		)
+	)
+	(label "Row 2"
+		(at 12.7 88.9 0)
+		(effects
+			(font
+				(size 1.27 1.27)
+			)
+			(justify left bottom)
+		)
+	)
+	(label "COL8"
+		(at 332.74 121.92 0)
+		(effects
+			(font
+				(size 1.27 1.27)
+			)
+			(justify left bottom)
+		)
+	)
+	(label "COL0"
+		(at 27.94 17.78 0)
+		(effects
+			(font
+				(size 1.27 1.27)
+			)
+			(justify left bottom)
+		)
+	)
 	(label "Row 5"
 		(at 332.74 124.46 0)
 		(effects
 			(font
-				(size 1.27 1.27)
-			)
-			(justify left bottom)
-		)
-	)
-	(label "COL12"
-		(at 218.44 17.78 0)
-		(effects
-			(font
-				(size 1.27 1.27)
-			)
-			(justify left bottom)
-		)
-	)
-	(label "COL14"
-		(at 243.84 17.78 0)
-		(effects
-			(font
-				(size 1.27 1.27)
-			)
-			(justify left bottom)
-		)
-	)
-	(label "Fn Row"
-		(at 332.74 86.36 0)
-		(effects
-			(font
-				(size 1.27 1.27)
-			)
-			(justify left bottom)
-		)
-	)
-	(label "COL5"
-		(at 332.74 114.3 0)
-		(effects
-			(font
-				(size 1.27 1.27)
-			)
-			(justify left bottom)
-		)
-	)
-	(label "COL11"
-		(at 392.43 91.44 0)
-		(effects
-			(font
-				(size 1.27 1.27)
-			)
-			(justify left bottom)
-		)
-	)
-	(label "COL10"
-		(at 193.04 17.78 0)
-		(effects
-			(font
-				(size 1.27 1.27)
-			)
-			(justify left bottom)
-		)
-	)
-	(label "COL13"
-		(at 392.43 96.52 0)
-		(effects
-			(font
-				(size 1.27 1.27)
-			)
-			(justify left bottom)
-		)
-	)
-	(label "COL12"
-		(at 392.43 93.98 0)
-		(effects
-			(font
-				(size 1.27 1.27)
-			)
-			(justify left bottom)
-		)
-	)
-	(label "Row 2"
-		(at 12.7 88.9 0)
-		(effects
-			(font
-				(size 1.27 1.27)
-			)
-			(justify left bottom)
-		)
-	)
-	(label "COL8"
-		(at 332.74 121.92 0)
-		(effects
-			(font
-				(size 1.27 1.27)
-			)
-			(justify left bottom)
-		)
-	)
-	(label "COL0"
-		(at 27.94 17.78 0)
-		(effects
-			(font
